Commit message: 仿真优化

File: src/robmini_description/urdf/lidar_gazebo.xacro (robot description, xacro)
@@ -29,5 +29,5 @@
                 <plugin name="gazebo_rplidar" filename="libgazebo_ros_ray_sensor.so">
                     <ros>
-                        <namespace>${tf_prefix}</namespace>    <!-- <namespace>${tf_prefix}</namespace>  -->
+                        <namespace>${ros_namespace}</namespace>
                         <remapping>~/out:=scan</remapping>
                     </ros>

File: src/robmini_description/urdf/robmini.ros2_control.xacro (robot description, xacro)
@@ -1,64 +1,75 @@
 <?xml version="1.0"?>
 <robot xmlns:xacro="http://www.ros.org/wiki/xacro" name="robmini">
-    <xacro:macro name="robmini_ros2_control" params="use_mock_bool:='false'">
-        <!-- <ros2_control name="robmini_hardware_interface" type="system"> -->
-        <ros2_control name="${'mecanum_mock_system' if use_mock_bool else 'mecanum_hw_system'}"
-                type="system">
-            <hardware>
-                <!-- <plugin>gazebo_ros2_control/GazeboSystem</plugin> -->
-                <plugin>${'mock_components/GenericSystem' if use_mock_bool else 'mecanum_hw_interface/MecanumHWSystem'}</plugin>
-                <xacro:if value="${use_mock_bool}">
-                    <!-- 关键：命令回灌到状态，mock 下就能看到运动了 -->
-                    <param name="fake_sensor_commands">true</param>
-                </xacro:if>
-                <xacro:unless value="${use_mock_bool}">
-                    <param name="device">/dev/ttySTM32</param>
-                    <param name="baud">115200</param>
-                </xacro:unless>
-            </hardware>
-            <joint name="front_left_wheel_joint">
-                <command_interface name="velocity">
-                    <param name="min">-10</param>
-                    <param name="max">10</param>
-                </command_interface>
-                <state_interface name="position" />
-                <state_interface name="velocity" />
-            </joint>
-            <joint name="front_right_wheel_joint">
-                <command_interface name="velocity">
-                    <param name="min">-10</param>
-                    <param name="max">10</param>
-                </command_interface>
-                <state_interface name="position" />
-                <state_interface name="velocity" />
-            </joint>
-            <joint name="rear_right_wheel_joint">
-                <command_interface name="velocity">
-                    <param name="min">-10</param>
-                    <param name="max">10</param>
-                </command_interface>
-                <state_interface name="position" />
-                <state_interface name="velocity" />
-            </joint>
-            <joint name="rear_left_wheel_joint">
-                <command_interface name="velocity">
-                    <param name="min">-10</param>
-                    <param name="max">10</param>
-                </command_interface>
-                <state_interface name="position" />
-                <state_interface name="velocity" />
-            </joint>
-        </ros2_control>
-        <!-- <gazebo>
-            <plugin name="gazebo_ros2_control" filename="libgazebo_ros2_control.so">
-                <update_rate>50</update_rate>
-                <parameters>$(find robmini_description)/config/robmini_mecanum_controllers.yaml</parameters>
-                <ros>
-                    <remapping>/robmini/mecanum_drive_controller_test01/tf_odometry:=/tf</remapping>
-                    <remapping>/robmini/mecanum_drive_controller_test01/reference_unstamped:=/robmini/cmd_vel</remapping>
-                    <remapping>/robmini/mecanum_drive_controller_test01/odometry:=/robmini/odom</remapping>
-                </ros>
-            </plugin>
-        </gazebo> -->
-    </xacro:macro>
+  <xacro:macro
+    name="robmini_ros2_control"
+    params="use_mock_bool:='false' use_gazebo_bool:='false' controller_config:='' ros_namespace:=''">
+    <ros2_control
+      name="${'mecanum_gazebo_system' if use_gazebo_bool else ('mecanum_mock_system' if use_mock_bool else 'mecanum_hw_system')}"
+      type="system">
+      <hardware>
+        <plugin>${'gazebo_ros2_control/GazeboSystem' if use_gazebo_bool else ('mock_components/GenericSystem' if use_mock_bool else 'mecanum_hw_interface/MecanumHWSystem')}</plugin>
+        <xacro:if value="${use_mock_bool and not use_gazebo_bool}">
+          <param name="fake_sensor_commands">true</param>
+        </xacro:if>
+        <!-- 除非在跑假测试或跑仿真，否则就执行下面代码 -->
+        <xacro:unless value="${use_mock_bool or use_gazebo_bool}">
+          <param name="device">/dev/ttySTM32</param>
+          <param name="baud">115200</param>
+        </xacro:unless>
+      </hardware>
+      <joint name="front_left_wheel_joint">
+        <command_interface name="velocity">
+          <param name="min">-10</param>
+          <param name="max">10</param>
+        </command_interface>
+        <state_interface name="position" />
+        <state_interface name="velocity" />
+      </joint>
+      <joint name="front_right_wheel_joint">
+        <command_interface name="velocity">
+          <param name="min">-10</param>
+          <param name="max">10</param>
+        </command_interface>
+        <state_interface name="position" />
+        <state_interface name="velocity" />
+      </joint>
+      <joint name="rear_right_wheel_joint">
+        <command_interface name="velocity">
+          <param name="min">-10</param>
+          <param name="max">10</param>
+        </command_interface>
+        <state_interface name="position" />
+        <state_interface name="velocity" />
+      </joint>
+      <joint name="rear_left_wheel_joint">
+        <command_interface name="velocity">
+          <param name="min">-10</param>
+          <param name="max">10</param>
+        </command_interface>
+        <state_interface name="position" />
+        <state_interface name="velocity" />
+      </joint>
+    </ros2_control>
+    <xacro:if value="${use_gazebo_bool}">
+    <xacro:property
+        name="topic_ns"
+        value="${'/' + ros_namespace if ros_namespace != '' else ''}" />
+    <gazebo>
+        <plugin filename="libgazebo_ros2_control.so" name="gazebo_ros2_control">
+        <ros>
+            <namespace>${ros_namespace}</namespace>
+            <!-- 把控制器发布的 TF 接到全局 /tf，否则 Nav2 看不到 odom -> base_link -->
+            <remapping>${topic_ns}/mecanum_drive_controller/tf_odometry:=/tf</remapping>
+            <!-- 把控制器里程计话题接到 Nav2 常用的 /robmini/odom -->
+            <remapping>${topic_ns}/mecanum_drive_controller/odometry:=${topic_ns}/odom</remapping>
+            <!-- 把 Nav2 输出的 /robmini/cmd_vel 接到 mecanum 控制器输入 -->
+            <remapping>${topic_ns}/mecanum_drive_controller/reference_unstamped:=${topic_ns}/cmd_vel</remapping>
+        </ros>
+        <xacro:if value="${controller_config != ''}">
+            <parameters>${controller_config}</parameters>
+        </xacro:if>
+        </plugin>
+    </gazebo>
+    </xacro:if>
+  </xacro:macro>
 </robot>

File: src/robmini_description/urdf/robmini.urdf.xacro (robot description, xacro)
@@ -1,4 +1,5 @@
 <?xml version="1.0" encoding="utf-8"?>
 <robot xmlns:xacro="http://www.ros.org/wiki/xacro">
+  <xacro:property name="mesh_dir" value="file://$(find robmini_description)/meshes" />
   <!-- <link name="${tf_prefix}base_footprint" />
         <joint name="base_joint" type="fixed">
@@ -28,6 +29,5 @@
         rpy="0 0 0" />
       <geometry>
-        <mesh
-          filename="package://robmini_description/meshes/base_link.STL" />
+        <mesh filename="${mesh_dir}/base_link.STL" />
         <!-- <mesh
           filename="file:///home/ksnc/robotmini_ws/src/robmini_description/meshes/base_link.STL" /> -->
@@ -44,6 +44,5 @@
         rpy="0 0 0" />
       <geometry>
-        <mesh
-          filename="package://robmini_description/meshes/base_link.STL" />
+        <mesh filename="${mesh_dir}/base_link.STL" />
         <!-- <mesh
           filename="file:///home/ksnc/robotmini_ws/src/robmini_description/meshes/base_link.STL" /> -->
@@ -72,6 +71,5 @@
         rpy="0 0 0" />
       <geometry>
-        <mesh
-          filename="package://robmini_description/meshes/left_front_wheel_link.STL" />
+        <mesh filename="${mesh_dir}/left_front_wheel_link.STL" />
         <!-- <mesh
           filename="file:///home/ksnc/robotmini_ws/src/robmini_description/meshes/left_front_wheel_link.STL" /> -->
@@ -88,6 +86,5 @@
         rpy="0 0 0" />
       <geometry>
-        <mesh
-          filename="package://robmini_description/meshes/left_front_wheel_link.STL" />
+        <mesh filename="${mesh_dir}/left_front_wheel_link.STL" />
         <!-- <mesh
           filename="file:///home/ksnc/robotmini_ws/src/robmini_description/meshes/left_front_wheel_link.STL" /> -->
@@ -129,6 +126,5 @@
         rpy="0 0 0" />
       <geometry>
-        <mesh
-          filename="package://robmini_description/meshes/left_back_wheel_link.STL" />
+        <mesh filename="${mesh_dir}/left_back_wheel_link.STL" />
         <!-- <mesh
           filename="file:///home/ksnc/robotmini_ws/src/robmini_description/meshes/left_back_wheel_link.STL" /> -->
@@ -145,6 +141,5 @@
         rpy="0 0 0" />
       <geometry>
-        <mesh
-          filename="package://robmini_description/meshes/left_back_wheel_link.STL" />
+        <mesh filename="${mesh_dir}/left_back_wheel_link.STL" />
         <!-- <mesh
           filename="file:///home/ksnc/robotmini_ws/src/robmini_description/meshes/left_back_wheel_link.STL" /> -->
@@ -186,6 +181,5 @@
         rpy="0 0 0" />
       <geometry>
-        <mesh
-          filename="package://robmini_description/meshes/right_back_wheel_link.STL" />
+        <mesh filename="${mesh_dir}/right_back_wheel_link.STL" />
         <!-- <mesh
           filename="file:///home/ksnc/robotmini_ws/src/robmini_description/meshes/right_back_wheel_link.STL" /> -->
@@ -202,6 +196,5 @@
         rpy="0 0 0" />
       <geometry>
-        <mesh
-          filename="package://robmini_description/meshes/right_back_wheel_link.STL" />
+        <mesh filename="${mesh_dir}/right_back_wheel_link.STL" />
         <!-- <mesh
           filename="file:///home/ksnc/robotmini_ws/src/robmini_description/meshes/right_back_wheel_link.STL" /> -->
@@ -243,6 +236,5 @@
         rpy="0 0 0" />
       <geometry>
-        <mesh
-          filename="package://robmini_description/meshes/right_front_wheel_link.STL" />
+        <mesh filename="${mesh_dir}/right_front_wheel_link.STL" />
         <!-- <mesh
           filename="file:///home/ksnc/robotmini_ws/src/robmini_description/meshes/right_front_wheel_link.STL" /> -->
@@ -259,6 +251,5 @@
         rpy="0 0 0" />
       <geometry>
-        <mesh
-          filename="package://robmini_description/meshes/right_front_wheel_link.STL" />
+        <mesh filename="${mesh_dir}/right_front_wheel_link.STL" />
         <!-- <mesh
           filename="file:///home/ksnc/robotmini_ws/src/robmini_description/meshes/right_front_wheel_link.STL" /> -->
@@ -300,6 +291,5 @@
         rpy="0 0 0" />
       <geometry>
-        <mesh
-          filename="package://robmini_description/meshes/lidar_link.STL" />
+        <mesh filename="${mesh_dir}/lidar_link.STL" />
         <!-- <mesh
           filename="file:///home/ksnc/robotmini_ws/src/robmini_description/meshes/lidar_link.STL" /> -->
@@ -316,6 +306,5 @@
         rpy="0 0 0" />
       <geometry>
-        <mesh
-          filename="package://robmini_description/meshes/lidar_link.STL" />
+        <mesh filename="${mesh_dir}/lidar_link.STL" />
         <!-- <mesh
           filename="file:///home/ksnc/robotmini_ws/src/robmini_description/meshes/lidar_link.STL" /> -->

File: src/robmini_description/urdf/robmini_run.urdf.xacro (robot description, xacro)
@@ -3,8 +3,14 @@
     <!-- 添加参数声明 -->
     <xacro:arg name="prefix" default=""/>
+    <xacro:arg name="namespace" default=""/>
     <xacro:arg name="use_mock" default="false"/>
+    <xacro:arg name="use_gazebo" default="false"/>
+    <xacro:arg name="controller_config" default=""/>
     <!-- 获取参数值 -->
     <xacro:property name="prefix" value="$(arg prefix)" />
-    <xacro:property name="use_mock" value="$(arg use_mock)"/>
+    <xacro:property name="ros_namespace" value="$(arg namespace)" />
+    <xacro:property name="use_mock" value="$(arg use_mock)" />
+    <xacro:property name="use_gazebo" value="$(arg use_gazebo)" />
+    <xacro:property name="controller_config" value="$(arg controller_config)" />
     <!-- TF 前缀处理保持不变 -->
     <xacro:if value="${prefix == '/' or prefix == '' or prefix == ' '}">
@@ -21,4 +27,7 @@
     <!-- <robmini/> -->
     <xacro:robmini_ros2_control
-      use_mock_bool="${str(use_mock).lower() in ['true','1','yes','on']}"/>
+    use_mock_bool="${str(use_mock).lower() in ['true', '1', 'yes', 'on']}"
+    use_gazebo_bool="${str(use_gazebo).lower() in ['true', '1', 'yes', 'on']}"
+    controller_config="${controller_config}"
+    ros_namespace="${ros_namespace}" />
 </robot>
