Commit message: 仿真兼容planar

File: src/robmini_description/urdf/robmini.ros2_control.xacro (robot description, xacro)
@@ -3,11 +3,19 @@
   <xacro:macro
     name="robmini_ros2_control"
-    params="use_mock_bool:='false' use_gazebo_bool:='false' controller_config:='' ros_namespace:=''">
+    params="use_mock_bool:='false' use_gazebo_bool:='false' sim_drive_mode:='planar' controller_config:='' ros_namespace:='' frame_prefix:=''">
+    <xacro:property
+      name="use_gazebo_ros2_control"
+      value="${use_gazebo_bool and sim_drive_mode == 'ros2_control'}" />
+    <xacro:property
+      name="use_gazebo_planar_move"
+      value="${use_gazebo_bool and sim_drive_mode == 'planar'}" />
+    <!-- 如果 use_gazebo_planar_move 这个变量的值是 False，那就执行下面代码 -->
+    <xacro:unless value="${use_gazebo_planar_move}">
     <ros2_control
-      name="${'mecanum_gazebo_system' if use_gazebo_bool else ('mecanum_mock_system' if use_mock_bool else 'mecanum_hw_system')}"
+      name="${'mecanum_gazebo_system' if use_gazebo_ros2_control else ('mecanum_mock_system' if use_mock_bool else 'mecanum_hw_system')}"
       type="system">
       <hardware>
-        <plugin>${'gazebo_ros2_control/GazeboSystem' if use_gazebo_bool else ('mock_components/GenericSystem' if use_mock_bool else 'mecanum_hw_interface/MecanumHWSystem')}</plugin>
-        <xacro:if value="${use_mock_bool and not use_gazebo_bool}">
+        <plugin>${'gazebo_ros2_control/GazeboSystem' if use_gazebo_ros2_control else ('mock_components/GenericSystem' if use_mock_bool else 'mecanum_hw_interface/MecanumHWSystem')}</plugin>
+        <xacro:if value="${use_mock_bool and not use_gazebo_ros2_control}">
           <param name="fake_sensor_commands">true</param>
         </xacro:if>
@@ -51,5 +59,6 @@
       </joint>
     </ros2_control>
-    <xacro:if value="${use_gazebo_bool}">
+    </xacro:unless>
+    <xacro:if value="${use_gazebo_ros2_control}">
     <xacro:property
         name="topic_ns"
@@ -72,4 +81,25 @@
     </gazebo>
     </xacro:if>
+    <xacro:if value="${use_gazebo_planar_move}">
+    <gazebo>
+        <plugin filename="libgazebo_ros_planar_move.so" name="gazebo_ros_planar_move">
+        <ros>
+            <namespace>${ros_namespace}</namespace>
+            <remapping>cmd_vel:=cmd_vel</remapping>
+            <remapping>odom:=odom</remapping>
+            <remapping>tf:=/tf</remapping>
+        </ros>
+        <update_rate>100</update_rate>
+        <publish_rate>50</publish_rate>
+        <publish_odom>true</publish_odom>
+        <publish_odom_tf>true</publish_odom_tf>
+        <odometry_frame>${frame_prefix}odom</odometry_frame>
+        <robot_base_frame>${frame_prefix}base_link</robot_base_frame>
+        <covariance_x>0.001</covariance_x>
+        <covariance_y>0.001</covariance_y>
+        <covariance_yaw>0.01</covariance_yaw>
+        </plugin>
+    </gazebo>
+    </xacro:if>
   </xacro:macro>
 </robot>

File: src/robmini_description/urdf/robmini.urdf.xacro (robot description, xacro)
@@ -2,4 +2,11 @@
 <robot xmlns:xacro="http://www.ros.org/wiki/xacro">
   <xacro:property name="mesh_dir" value="file://$(find robmini_description)/meshes" />
+  <xacro:property
+    name="use_planar_drive"
+    value="${str(use_gazebo).lower() in ['true', '1', 'yes', 'on'] and sim_drive_mode == 'planar'}" />
+  <xacro:property name="planar_wheel_collision_radius" value="0.04" />
+  <xacro:property name="wheel_ground_mu" value="${0.02 if use_planar_drive else 1.5}" />
+  <xacro:property name="wheel_ground_mu2" value="${0.02 if use_planar_drive else 1.2}" />
+  <xacro:property name="wheel_ground_slip" value="${1.0 if use_planar_drive else 0.0}" />
   <!-- <link name="${tf_prefix}base_footprint" />
         <joint name="base_joint" type="fixed">
@@ -86,7 +93,12 @@
         rpy="0 0 0" />
       <geometry>
-        <mesh filename="${mesh_dir}/left_front_wheel_link.STL" />
-        <!-- <mesh
-          filename="file:///home/ksnc/robotmini_ws/src/robmini_description/meshes/left_front_wheel_link.STL" /> -->
+        <xacro:if value="${use_planar_drive}">
+          <sphere radius="${planar_wheel_collision_radius}" />
+        </xacro:if>
+        <xacro:unless value="${use_planar_drive}">
+          <mesh filename="${mesh_dir}/left_front_wheel_link.STL" />
+          <!-- <mesh
+            filename="file:///home/ksnc/robotmini_ws/src/robmini_description/meshes/left_front_wheel_link.STL" /> -->
+        </xacro:unless>
       </geometry>
     </collision>
@@ -141,7 +153,12 @@
         rpy="0 0 0" />
       <geometry>
-        <mesh filename="${mesh_dir}/left_back_wheel_link.STL" />
-        <!-- <mesh
-          filename="file:///home/ksnc/robotmini_ws/src/robmini_description/meshes/left_back_wheel_link.STL" /> -->
+        <xacro:if value="${use_planar_drive}">
+          <sphere radius="${planar_wheel_collision_radius}" />
+        </xacro:if>
+        <xacro:unless value="${use_planar_drive}">
+          <mesh filename="${mesh_dir}/left_back_wheel_link.STL" />
+          <!-- <mesh
+            filename="file:///home/ksnc/robotmini_ws/src/robmini_description/meshes/left_back_wheel_link.STL" /> -->
+        </xacro:unless>
       </geometry>
     </collision>
@@ -196,7 +213,12 @@
         rpy="0 0 0" />
       <geometry>
-        <mesh filename="${mesh_dir}/right_back_wheel_link.STL" />
-        <!-- <mesh
-          filename="file:///home/ksnc/robotmini_ws/src/robmini_description/meshes/right_back_wheel_link.STL" /> -->
+        <xacro:if value="${use_planar_drive}">
+          <sphere radius="${planar_wheel_collision_radius}" />
+        </xacro:if>
+        <xacro:unless value="${use_planar_drive}">
+          <mesh filename="${mesh_dir}/right_back_wheel_link.STL" />
+          <!-- <mesh
+            filename="file:///home/ksnc/robotmini_ws/src/robmini_description/meshes/right_back_wheel_link.STL" /> -->
+        </xacro:unless>
       </geometry>
     </collision>
@@ -251,7 +273,12 @@
         rpy="0 0 0" />
       <geometry>
-        <mesh filename="${mesh_dir}/right_front_wheel_link.STL" />
-        <!-- <mesh
-          filename="file:///home/ksnc/robotmini_ws/src/robmini_description/meshes/right_front_wheel_link.STL" /> -->
+        <xacro:if value="${use_planar_drive}">
+          <sphere radius="${planar_wheel_collision_radius}" />
+        </xacro:if>
+        <xacro:unless value="${use_planar_drive}">
+          <mesh filename="${mesh_dir}/right_front_wheel_link.STL" />
+          <!-- <mesh
+            filename="file:///home/ksnc/robotmini_ws/src/robmini_description/meshes/right_front_wheel_link.STL" /> -->
+        </xacro:unless>
       </geometry>
     </collision>
@@ -369,7 +396,9 @@
         <friction>
             <ode>
-            <mu>1.5</mu>
-            <mu2>1.2</mu2>
+            <mu>${wheel_ground_mu}</mu>
+            <mu2>${wheel_ground_mu2}</mu2>
             <fdir1>1 -1 0</fdir1>
+            <slip1>${wheel_ground_slip}</slip1>
+            <slip2>${wheel_ground_slip}</slip2>
             </ode>
         </friction>
@@ -382,7 +411,9 @@
         <friction>
             <ode>
-            <mu>1.5</mu>
-            <mu2>1.2</mu2>
+            <mu>${wheel_ground_mu}</mu>
+            <mu2>${wheel_ground_mu2}</mu2>
             <fdir1>1 1 0</fdir1>
+            <slip1>${wheel_ground_slip}</slip1>
+            <slip2>${wheel_ground_slip}</slip2>
             </ode>
         </friction>
@@ -395,7 +426,9 @@
         <friction>
             <ode>
-            <mu>1.5</mu>
-            <mu2>1.2</mu2>
+            <mu>${wheel_ground_mu}</mu>
+            <mu2>${wheel_ground_mu2}</mu2>
             <fdir1>1 1 0</fdir1>
+            <slip1>${wheel_ground_slip}</slip1>
+            <slip2>${wheel_ground_slip}</slip2>
             </ode>
         </friction>
@@ -408,7 +441,9 @@
         <friction>
             <ode>
-            <mu>1.5</mu>
-            <mu2>1.2</mu2>
+            <mu>${wheel_ground_mu}</mu>
+            <mu2>${wheel_ground_mu2}</mu2>
             <fdir1>1 -1 0</fdir1>
+            <slip1>${wheel_ground_slip}</slip1>
+            <slip2>${wheel_ground_slip}</slip2>
             </ode>
         </friction>

File: src/robmini_description/urdf/robmini_run.urdf.xacro (robot description, xacro)
@@ -6,4 +6,5 @@
     <xacro:arg name="use_mock" default="false"/>
     <xacro:arg name="use_gazebo" default="false"/>
+    <xacro:arg name="sim_drive_mode" default="planar"/>  <!-- /ros2_control-->
     <xacro:arg name="controller_config" default=""/>
     <!-- 获取参数值 -->
@@ -12,4 +13,5 @@
     <xacro:property name="use_mock" value="$(arg use_mock)" />
     <xacro:property name="use_gazebo" value="$(arg use_gazebo)" />
+    <xacro:property name="sim_drive_mode" value="$(arg sim_drive_mode)" />
     <xacro:property name="controller_config" value="$(arg controller_config)" />
     <!-- TF 前缀处理保持不变 -->
@@ -29,5 +31,7 @@
     use_mock_bool="${str(use_mock).lower() in ['true', '1', 'yes', 'on']}"
     use_gazebo_bool="${str(use_gazebo).lower() in ['true', '1', 'yes', 'on']}"
+    sim_drive_mode="${sim_drive_mode}"
     controller_config="${controller_config}"
-    ros_namespace="${ros_namespace}" />
+    ros_namespace="${ros_namespace}"
+    frame_prefix="${tf_prefix}" />
 </robot>
