Commit message: 实车测试

File: src/robmini_description/urdf/robmini.urdf.xacro (robot description, xacro)
@@ -1,5 +1,6 @@
 <?xml version="1.0" encoding="utf-8"?>
 <robot xmlns:xacro="http://www.ros.org/wiki/xacro">
-  <xacro:property name="mesh_dir" value="file://$(find robmini_description)/meshes" />
+  <!-- file://$(find robmini_description)/meshes -->
+  <xacro:property name="mesh_dir" value="package://robmini_description/meshes" />
   <xacro:property
     name="use_planar_drive"

Commit message: 小更新

File: src/robmini_description/urdf/robmini.urdf.xacro (robot description, xacro)
@@ -1,6 +1,6 @@
 <?xml version="1.0" encoding="utf-8"?>
 <robot xmlns:xacro="http://www.ros.org/wiki/xacro">
-  <!-- file://$(find robmini_description)/meshes -->
-  <xacro:property name="mesh_dir" value="package://robmini_description/meshes" />
+  <!-- <xacro:property name="mesh_dir" value="package://robmini_description/meshes" /> -->
+  <xacro:property name="mesh_dir" value="file://$(find robmini_description)/meshes" />
   <xacro:property
     name="use_planar_drive"
